File: ip175.kicad_pcb (KiCad board)
At the start: 2 copper layers, 73.7 x 43.2 mm, 56 parts, among them J1 Conn_02x10_Counter_Clockwise, J2 Conn_02x10_Counter_Clockwise, J3 Conn_02x10_Counter_Clockwise, J4 Conn_01x02_Male, J5 Conn_01x02_Male, J6 Conn_01x02_Male, U1 ip175, U2 at24c16, U3 AMS1117-3.3, Y1 25MHz

Commit message: Закончили разводку платы, отправили в производство
Parts:
- moved R2 4.09 mm to (153.3, 96.2)
- moved TR2 3.69 mm to (145.1, 93.6)
- moved C5 3.53 mm to (153.0, 92.1)
- moved C2 3.20 mm to (136.4, 91.7)
- moved C14 2.62 mm to (184.7, 78.2), turned to 180 degrees
- moved U1 2.50 mm to (167.9, 87.2)
- moved R1 2.27 mm to (134.9, 95.8), turned to 0 degrees
- moved C13 2.16 mm to (178.6, 78.2), turned to 0 degrees
- moved R8 2.09 mm to (185.4, 95.8)
- moved C9 2.09 mm to (182.4, 93.5)
- moved C7 2.09 mm to (187.7, 95.5)
- moved C8 2.09 mm to (187.7, 91.2)
- moved ETH3_RX 2.09 mm to (191.3, 94.5)
- moved R9 2.09 mm to (185.4, 90.9)
- moved R22 1.84 mm to (156.2, 81.2)
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- renumbered J1 to ETH0, J2 to ETH1, J3 to ETH2, J4 to ETH3_RX, J5 to ETH3_TX, D1 to LINK0, D2 to LINK1, D3 to LINK2, D4 to LINK3, D5 to LINK4, J6 to POWER, D6 to VLAN
Connections:
- U1 pad 1: Net-(TR2-Pad3) -> Net-(TR2-Pad8)
- U1 pad 10: Net-(TR3-Pad1) -> Net-(TR3-Pad3)
- U1 pad 11: Net-(TR3-Pad3) -> Net-(TR3-Pad1)
- U1 pad 2: Net-(TR2-Pad1) -> Net-(TR2-Pad6)
- U1 pad 3: Net-(TR2-Pad8) -> Net-(TR2-Pad3)
- U1 pad 4: Net-(TR2-Pad6) -> Net-(TR2-Pad1)
- U1 pad 44: Net-(TR1-Pad6) -> Net-(TR1-Pad8)
- U1 pad 45: Net-(TR1-Pad8) -> Net-(TR1-Pad6)
- U1 pad 46: Net-(TR1-Pad1) -> Net-(TR1-Pad3)
- U1 pad 47: Net-(TR1-Pad3) -> Net-(TR1-Pad1)
- U1 pad 8: Net-(TR3-Pad6) -> Net-(TR3-Pad8)
- U1 pad 9: Net-(TR3-Pad8) -> Net-(TR3-Pad6)
Routing:
- net +3V3: track 121.8 -> 167.8 mm, vias 6 -> 8
- net Net-(J3-Pad3): track 58.2 -> 35.1 mm
- net Net-(J3-Pad4): track 35.7 -> 44.2 mm
- net Net-(TR2-Pad8): track 34.3 -> 28.2 mm, vias 2 -> 0
- net Net-(TR2-Pad6): track 32.3 -> 26.4 mm, vias 2 -> 0
- net Net-(R11-Pad1): track 24.5 -> 30.2 mm, vias 3 -> 2
- net Net-(R18-Pad2): track 20.2 -> 25.3 mm
- net Net-(R11-Pad2): track 16.2 -> 21.0 mm
- net Net-(C2-Pad1): track 18.2 -> 21.9 mm
- net Net-(J2-Pad3): track 12.9 -> 9.30 mm
- net Net-(J2-Pad2): track 11.6 -> 8.03 mm
- net Net-(J2-Pad1): track 11.6 -> 8.03 mm
- net Net-(J2-Pad4): track 12.8 -> 9.30 mm
- net Net-(TR3-Pad1): track 9.97 -> 7.04 mm, vias 2 -> 0
- net Net-(TR2-Pad1): track 22.9 -> 20.0 mm
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- added copper zone on B.Cu, net GND
- added copper zone on F.Cu, net GND
Other:
- board size 73.7 x 43.2 mm -> 72.6 x 43.2 mm
- net class +3 added: clearance 0.2, trace_width 0.4, via_dia 0.8, via_drill 0.4
- net class +5 added: clearance 0.2, trace_width 1, via_dia 0.8, via_drill 0.4
- board text added: "+5"
- board text added: "-"
