File: ip175.sch (KiCad schematic (older format))
At the start: 51 parts

Commit message: Закончили со схемой (нужно перепроверить) + предварительная разводка платы
Parts:
- added J2, J3: Conn_02x10_Counter_Clockwise, ip175:FR_Conn, symbol Connector_Generic:Conn_02x10_Counter_Clockwise
- added J4, J5, J6: Conn_01x02_Male, kicadgithub:PinHeader_1x02_P2.54mm_Vertical, symbol Connector:Conn_01x02_Male
- C1, C10, C11, C12, C13, C14, C15, C2, C3, C4, C5, C6, C7, C8, C9: renamed from C?; footprint (none) -> kicadgithub:C_0805_2012Metric_Pad1.18x1.45mm_HandSolder
- D1, D2, D3, D4, D5, D6: renamed from D?; footprint (none) -> kicadgithub:LED_0805_2012Metric_Pad1.15x1.40mm_HandSolder
- J1: renamed from J?; footprint (none) -> ip175:FR_Conn
- R1, R10, R11, R12, R13, R14, R15, R16, R17, R18, R19, R2, R20, R21, R22, R3, R4, R5, R6, R7, R8, R9: renamed from R?; footprint (none) -> kicadgithub:R_0603_1608Metric_Pad0.98x0.95mm_HandSolder
- TR1, TR2, TR3: renamed from TR?; footprint Transformer_SMD:Transformer_Ethernet_Bourns_PT61017PEL -> kicadgithub:Transformer_Ethernet_Bourns_PT61017PEL
- U1: renamed from U?; footprint (none) -> kicadgithub:QFN-48-1EP_6x6mm_P0.4mm_EP4.2x4.2mm_ThermalVias
- U2: renamed from U?; footprint (none) -> kicadgithub:SOIC-8_3.9x4.9mm_P1.27mm
- U3: renamed from U?; footprint Package_TO_SOT_SMD:SOT-223-3_TabPin2 -> kicadgithub:SOT-223-3_TabPin2
- Y1: renamed from Y?; footprint (none) -> kicadgithub:Crystal_SMD_HC49-SD
Connections:
- net +5V: now also J1.8 (Pin_8), J2.8 (Pin_8), J3.8 (Pin_8), J6.2 (Pin_2)
- net GND: now also J1.5 (Pin_5), J2.5 (Pin_5), J3.5 (Pin_5), J6.1 (Pin_1)
- net at R9.2, U1.15 (RXI3-): now also C8.1; no longer C8.2
- net at R10.2, U1.16 (TXO3+): now also C11.1; no longer C11.2
- net at R12.2, U1.17 (TXO3-): now also C12.1; no longer C12.2
- net at TR2.11 (RX+): now also J2.3 (Pin_3)
- net at TR2.14 (TX-): now also J2.2 (Pin_2)
- net at TR2.16 (TX+): now also J2.1 (Pin_1)
- net at TR2.9 (RX-): now also J2.4 (Pin_4)
- net at TR3.11 (RX+): now also J3.3 (Pin_3)
- net at TR3.14 (TX-): now also J3.2 (Pin_2)
- net at TR3.16 (TX+): now also J3.1 (Pin_1)
- net at TR3.9 (RX-): now also J3.4 (Pin_4)
- net at TR1.11 (RX+): now also J1.3 (Pin_3)
- net at TR1.14 (TX-): now also J1.2 (Pin_2)
- net at TR1.16 (TX+): now also J1.1 (Pin_1)
- net at TR1.9 (RX-): now also J1.4 (Pin_4)
- net at C7.1: now also J4.1 (Pin_1)
- new net: C8.2, J4.2 (Pin_2)
- new net: C12.2, J5.1 (Pin_1)
- new net: C11.2, J5.2 (Pin_2)
- no-connect marks 4 -> 46
Other:
- moved on the sheet: C11, C12, C7, C8, J1

Commit message: Закончили разводку платы, отправили в производство
Connections:
- net at U1.1 (TXO1-): now also TR2.8 (RD-); no longer TR2.3 (TD-)
- net at U1.10 (TXO2+): now also TR3.3 (TD-); no longer TR3.1 (TD+)
- net at U1.11 (TXO2-): now also TR3.1 (TD+); no longer TR3.3 (TD-)
- net at U1.2 (TXO1+): now also TR2.6 (RD+); no longer TR2.1 (TD+)
- net at U1.3 (RXI1-): now also TR2.3 (TD-); no longer TR2.8 (RD-)
- net at U1.4 (RXI1+): now also TR2.1 (TD+); no longer TR2.6 (RD+)
- net at U1.44 (RXI0+): now also TR1.8 (RD-); no longer TR1.6 (RD+)
- net at U1.45 (RXI0-): now also TR1.6 (RD+); no longer TR1.8 (RD-)
- net at U1.46 (TXO0+): now also TR1.3 (TD-); no longer TR1.1 (TD+)
- net at U1.47 (TXO0-): now also TR1.1 (TD+); no longer TR1.3 (TD-)
- net at U1.8 (RXI2+): now also TR3.8 (RD-); no longer TR3.6 (RD+)
- net at U1.9 (RXI2-): now also TR3.6 (RD+); no longer TR3.8 (RD-)
Changed lines of the file:
@@
 $EndComp
-Wire Wire Line
-	3500 2900 4150 2900
-Wire Wire Line
-	4150 2900 4150 3500
 Wire Wire Line
 	4150 3500 4900 3500
 Wire Wire Line
-	3500 2700 4200 2700
-Wire Wire Line
-	4200 2700 4200 3400
+	3500 2700 3600 2700
 Wire Wire Line
 	4200 3400 4900 3400
-Wire Wire Line
-	4300 3700 4300 2500
-Wire Wire Line
-	4300 2500 3500 2500
-Wire Wire Line
-	4300 3700 4900 3700
-Wire Wire Line
-	3500 2300 4350 2300
-Wire Wire Line
-	4350 2300 4350 3600
-Wire Wire Line
-	4350 3600 4900 3600
 $Comp
 L Device:C_Small C5
@@
 $EndComp
 Wire Wire Line
-	4200 5000 4200 4200
-Wire Wire Line
-	4200 4200 4900 4200
-Wire Wire Line
-	3500 5000 4200 5000
-Wire Wire Line
 	4900 4100 4300 4100
 Wire Wire Line
-	4300 4100 4300 5200
-Wire Wire Line
-	4300 5200 3500 5200
-Wire Wire Line
-	3500 5400 4400 5400
-Wire Wire Line
-	4400 5400 4400 4400
-Wire Wire Line
-	4400 4400 4900 4400
-Wire Wire Line
 	4900 4300 4450 4300
-Wire Wire Line
-	4450 4300 4450 5600
-Wire Wire Line
-	4450 5600 3500 5600
 $Comp
 L Device:C_Small C6
@@
 	-1   0    0    -1
 $EndComp
-Wire Wire Line
-	3500 700  5750 700
-Wire Wire Line
-	5750 700  5750 2850
-Wire Wire Line
-	3500 900  5850 900
-Wire Wire Line
-	5850 900  5850 2850
-Wire Wire Line
-	3500 1100 5550 1100
-Wire Wire Line
-	5550 1100 5550 2850
-Wire Wire Line
-	3500 1300 5650 1300
-Wire Wire Line
-	5650 1300 5650 2850
 $Comp
 L Device:C_Small C4
@@
 Wire Wire Line
 	6150 6200 6150 6500
+Wire Wire Line
+	4300 5000 4300 4100
+Wire Wire Line
+	3500 5000 4300 5000
+Wire Wire Line
+	3500 5200 4150 5200
+Wire Wire Line
+	4150 5200 4150 4200
+Wire Wire Line
+	4150 4200 4900 4200
+Wire Wire Line
+	4350 4400 4900 4400
+Wire Wire Line
+	4450 4300 4450 5400
+Wire Wire Line
+	4450 5400 3500 5400
+Wire Wire Line
+	4350 4400 4350 5600
+Wire Wire Line
+	4350 5600 3500 5600
+Wire Wire Line
+	3500 2900 3500 3700
+Wire Wire Line
+	3500 3700 4900 3700
+Wire Wire Line
+	3600 3600 3600 2700
+Wire Wire Line
+	3500 2300 4200 2300
+Wire Wire Line
+	4200 2300 4200 3400
+Wire Wire Line
+	3500 2500 4150 2500
+Wire Wire Line
+	4150 2500 4150 3500
+Wire Wire Line
+	3600 3600 4900 3600
+Wire Wire Line
+	5650 1100 3500 1100
+Wire Wire Line
+	5650 1100 5650 2850
+Wire Wire Line
+	3500 1300 5550 1300
+Wire Wire Line
+	5550 1300 5550 2850
+Wire Wire Line
+	3500 700  5850 700
+Wire Wire Line
+	5850 700  5850 2850
+Wire Wire Line
+	5750 900  5750 2850
+Wire Wire Line
+	3500 900  5750 900
 $EndSCHEMATC
